File: board/misteryshield20k/misteryshield20k.kicad_sch (KiCad schematic)
At the start: 41 parts, among them J1 Joystick, J2 USB_C_Receptacle_USB2.0, J3 MIDI OUT, J4 MIDI IN, J5 Conn_02x06_Odd_Even, J6 Conn_01x20_Socket, J7 Conn_01x20_Socket, J8 Conn_02x04_Pin, Q1 BSS123, Q2 BSS123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

Commit message: Fix #38
Parts:
- R9: LCSC Part # C17530 -> C17590
Changed lines of the file:
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@@
       (effects (font (size 1.27 1.27)) hide)
     )
-    (property "LCSC Part #" " C17530" (at 131.445 117.475 0)
+    (property "LCSC Part #" " C17590" (at 131.445 117.475 0)
       (effects (font (size 1.27 1.27)) hide)
     )
