File: board/misteryshield20k/misteryshield20k_m0s.kicad_sch (KiCad schematic)
At the start: 38 parts, among them J1 Joystick, J3 MIDI OUT, J4 MIDI IN, J5 Conn_02x06_Odd_Even, J6 Conn_01x20_Socket, J7 Conn_01x20_Socket, J8 Conn_02x04_Pin, Q1 BSS123, Q2 BSS123, Q3 BSS123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

Commit message: Update production data
Parts:
- J1: JLCPCB Position Offset 1,5.5 -> 0,6
- J5: JLCPCB Position Offset 6.35,-1.5 -> 4.5,0
- J8: JLCPCB Position Offset -3.81,-1.27 -> (none)
